Commit message: redid URDF export and assemblies with the old orientations, but with the sizing and origins fixed

File: part_files/V4/Harold_URDF_Export_2/urdf/Harold_URDF_Export_2.urdf (robot description, URDF)
Before this commit: robot Harold_URDF_Export, 13 links, 12 joints
Links:
- link Body: mass 0.65516 -> 0.655160642240757; geometry collision mesh filename=package://Harold_URDF_Export_2/meshes/Body.STL; visual mesh filename=package://Harold_URDF_Export_2/meshes/Body.STL
- link bl_calf: geometry collision mesh filename=package://Harold_URDF_Export_2/meshes/bl_calf.STL; visual mesh filename=package://Harold_URDF_Export_2/meshes/bl_calf.STL
- link bl_shoulder: geometry collision mesh filename=package://Harold_URDF_Export_2/meshes/bl_shoulder.STL; visual mesh filename=package://Harold_URDF_Export_2/meshes/bl_shoulder.STL
- link bl_thigh: geometry collision mesh filename=package://Harold_URDF_Export_2/meshes/bl_thigh.STL; visual mesh filename=package://Harold_URDF_Export_2/meshes/bl_thigh.STL
- link br_calf: geometry collision mesh filename=package://Harold_URDF_Export_2/meshes/br_calf.STL; visual mesh filename=package://Harold_URDF_Export_2/meshes/br_calf.STL
- link br_shoulder: mass 0.0776965557993419 -> 0.0776965557993418; geometry collision mesh filename=package://Harold_URDF_Export_2/meshes/br_shoulder.STL; visual mesh filename=package://Harold_URDF_Export_2/meshes/br_shoulder.STL
- link br_thigh: geometry collision mesh filename=package://Harold_URDF_Export_2/meshes/br_thigh.STL; visual mesh filename=package://Harold_URDF_Export_2/meshes/br_thigh.STL
- link fl_calf: geometry collision mesh filename=package://Harold_URDF_Export_2/meshes/fl_calf.STL; visual mesh filename=package://Harold_URDF_Export_2/meshes/fl_calf.STL
- link fl_shoulder: geometry collision mesh filename=package://Harold_URDF_Export_2/meshes/fl_shoulder.STL; visual mesh filename=package://Harold_URDF_Export_2/meshes/fl_shoulder.STL
- link fl_thigh: geometry collision mesh filename=package://Harold_URDF_Export_2/meshes/fl_thigh.STL; visual mesh filename=package://Harold_URDF_Export_2/meshes/fl_thigh.STL
- link fr_calf: geometry collision mesh filename=package://Harold_URDF_Export_2/meshes/fr_calf.STL; visual mesh filename=package://Harold_URDF_Export_2/meshes/fr_calf.STL
- link fr_shoulder: mass 0.0776965557993419 -> 0.0776965557993418; geometry collision mesh filename=package://Harold_URDF_Export_2/meshes/fr_shoulder.STL; visual mesh filename=package://Harold_URDF_Export_2/meshes/fr_shoulder.STL
- link fr_thigh: geometry collision mesh filename=package://Harold_URDF_Export_2/meshes/fr_thigh.STL; visual mesh filename=package://Harold_URDF_Export_2/meshes/fr_thigh.STL
Joints:
- joint bl_calf_joint: origin xyz=0.0025 -0.10288 0.005 rpy=0 0 0 -> xyz=0.00249999999999997 -0.102875 0.00500000000000127 rpy=0 0 0
- joint br_calf_joint: origin xyz=0.0025 -0.10288 -0.005 rpy=0 0 0 -> xyz=0.0025 -0.102875 -0.00500000000000039 rpy=0 0 0
- joint br_shoulder_joint: origin xyz=0.1854 0.048 0.0175 rpy=1.5708 0 0 -> xyz=0.185399999999999 0.048 0.0175 rpy=1.5707963267949 0 0
- joint fl_calf_joint: origin xyz=0.0025 -0.10288 0.005 rpy=0 0 0 -> xyz=0.00249999999999997 -0.102875 0.00500000000000111 rpy=0 0 0
- joint fr_calf_joint: origin xyz=0.0025 -0.10288 -0.005 rpy=0 0 0 -> xyz=0.0025 -0.102875 -0.00500000000000027 rpy=0 0 0
- joint fr_thigh_joint: origin xyz=-0.0232 0.011125 -0.0101 rpy=0 0 0 -> xyz=-0.0232000000000001 0.011125 -0.0100999999999999 rpy=0 0 0
